Commit message: parametrize scheduling policy, if we want SLAVE async mode

File: ur_robot_driver/urdf/ur.ros2_control.xacro (robot description, xacro)
@@ -26,4 +26,5 @@
     robot_receive_timeout:=0.04
     rw_rate:=0
+    scheduling_policy:=''
     ">
     <!-- rw_rate of 0 uses the rate of the controller_manager -->
@@ -34,5 +35,11 @@
     <!--<xacro:ur_arm_transmission prefix="${prefix}" hw_interface="${transmission_hw_interface}" />-->
     <!-- Placeholder for ros2_control transmission which don't yet exist -->
-    <ros2_control name="${name}" type="system" rw_rate="${rw_rate}">
+    <xacro:property name="is_async" value="${use_mock_hardware == 0 and scheduling_policy != ''}"/>
+    <ros2_control name="${name}" type="system" rw_rate="${rw_rate}" is_async="${is_async}">
+      <xacro:if value="${is_async}">
+        <properties>
+          <async scheduling_policy="${scheduling_policy}" print_warnings="true" thread_priority="30"/>
+        </properties>
+      </xacro:if>
       <hardware>
         <xacro:if value="${use_mock_hardware}">

Commit message: parametrize scheduling policy, if we want SLAVE async mode

File: ur_robot_driver/urdf/ur.ros2_control.xacro (robot description, xacro)
@@ -29,4 +29,5 @@
     verify_robot_model:=false
     use_currents_as_efforts:=true
+    scheduling_policy:=''
     ">
     <!-- rw_rate of 0 uses the rate of the controller_manager -->
@@ -37,5 +38,11 @@
     <!--<xacro:ur_arm_transmission prefix="${prefix}" hw_interface="${transmission_hw_interface}" />-->
     <!-- Placeholder for ros2_control transmission which don't yet exist -->
-    <ros2_control name="${name}" type="system" rw_rate="${rw_rate}">
+    <xacro:property name="is_async" value="${use_mock_hardware == 0 and scheduling_policy != ''}"/>
+    <ros2_control name="${name}" type="system" rw_rate="${rw_rate}" is_async="${is_async}">
+      <xacro:if value="${is_async}">
+        <properties>
+          <async scheduling_policy="${scheduling_policy}" print_warnings="true" thread_priority="30"/>
+        </properties>
+      </xacro:if>
       <hardware>
         <xacro:if value="${use_mock_hardware}">

File: ur_robot_driver/urdf/ur.urdf.xacro (robot description, xacro)
@@ -35,4 +35,5 @@
   <xacro:arg name="blocking_read" default="false" />
   <xacro:arg name="rw_rate" default="0" />
+  <xacro:arg name="scheduling_policy" default="" />
   <!--   tool communication related parameters-->
   <xacro:arg name="use_tool_communication" default="false" />
@@ -103,4 +104,5 @@
     non_blocking_read="${not blocking_read}"
     rw_rate="$(arg rw_rate)"
+    scheduling_policy="$(arg scheduling_policy)"
   />
 </robot>

Commit message: parametrize scheduling policy, if we want SLAVE async mode

File: ur_robot_driver/urdf/ur.ros2_control.xacro (robot description, xacro)
@@ -28,4 +28,5 @@
     rw_rate:=0
     verify_robot_model:=false
+    scheduling_policy:=''
     ">
     <!-- rw_rate of 0 uses the rate of the controller_manager -->
@@ -36,5 +37,11 @@
     <!--<xacro:ur_arm_transmission prefix="${prefix}" hw_interface="${transmission_hw_interface}" />-->
     <!-- Placeholder for ros2_control transmission which don't yet exist -->
-    <ros2_control name="${name}" type="system" rw_rate="${rw_rate}">
+    <xacro:property name="is_async" value="${use_mock_hardware == 0 and scheduling_policy != ''}"/>
+    <ros2_control name="${name}" type="system" rw_rate="${rw_rate}" is_async="${is_async}">
+      <xacro:if value="${is_async}">
+        <properties>
+          <async scheduling_policy="${scheduling_policy}" print_warnings="true" thread_priority="30"/>
+        </properties>
+      </xacro:if>
       <hardware>
         <xacro:if value="${use_mock_hardware}">

File: ur_robot_driver/urdf/ur.urdf.xacro (robot description, xacro)
@@ -33,4 +33,5 @@
   <xacro:arg name="verify_robot_model" default="false" />
   <xacro:arg name="rw_rate" default="0" />
+  <xacro:arg name="scheduling_policy" default="" />
   <!--   tool communication related parameters-->
   <xacro:arg name="use_tool_communication" default="false" />
@@ -98,4 +99,5 @@
     verify_robot_model="$(arg verify_robot_model)"
     rw_rate="$(arg rw_rate)"
+    scheduling_policy="$(arg scheduling_policy)"
   />
 </robot>

Commit message: parametrize scheduling policy, if we want SLAVE async mode

File: ur_robot_driver/urdf/ur.ros2_control.xacro (robot description, xacro)
@@ -26,4 +26,5 @@
     robot_receive_timeout:=0.04
     rw_rate:=0
+    scheduling_policy:=''
     ">
     <!-- rw_rate of 0 uses the rate of the controller_manager -->
@@ -34,5 +35,11 @@
     <!--<xacro:ur_arm_transmission prefix="${prefix}" hw_interface="${transmission_hw_interface}" />-->
     <!-- Placeholder for ros2_control transmission which don't yet exist -->
-    <ros2_control name="${name}" type="system" rw_rate="${rw_rate}">
+    <xacro:property name="is_async" value="${use_mock_hardware == 0 and scheduling_policy != ''}"/>
+    <ros2_control name="${name}" type="system" rw_rate="${rw_rate}" is_async="${is_async}">
+      <xacro:if value="${is_async}">
+        <properties>
+          <async scheduling_policy="${scheduling_policy}" print_warnings="true" thread_priority="30"/>
+        </properties>
+      </xacro:if>
       <hardware>
         <xacro:if value="${use_mock_hardware}">

File: ur_robot_driver/urdf/ur.urdf.xacro (robot description, xacro)
@@ -32,4 +32,5 @@
   <xacro:arg name="trajectory_port" default="50003"/>
   <xacro:arg name="rw_rate" default="0" />
+  <xacro:arg name="scheduling_policy" default="" />
   <!--   tool communication related parameters-->
   <xacro:arg name="use_tool_communication" default="false" />
@@ -95,4 +96,5 @@
     trajectory_port="$(arg trajectory_port)"
     rw_rate="$(arg rw_rate)"
+    scheduling_policy="$(arg scheduling_policy)"
   />
 </robot>
